File: hardware/main-controller-v1/main-controller-v1.kicad_sch (KiCad schematic)
At the start: 59 parts, among them J1 USB_C_Receptacle_USB2.0_16P, J2 Screw_Terminal_01x02, J3 Screw_Terminal_01x02, J4 Screw_Terminal_01x02, J6 Screw_Terminal_01x14, K1 G3MB-202P, K10 G3MB-202P, K11 G3MB-202P, K12 G3MB-202P, K2 G3MB-202P, K3 G3MB-202P, K4 G3MB-202P, K5 G3MB-202P, K6 G3MB-202P, K7 G3MB-202P, K8 G3MB-202P, K9 G3MB-202P, SW1 SW_Push, SW2 SW_Push, U1 ESP32-S3-WROOM-1, U2 USBLC6-2SC6, U3 LM2596S-5, U4 AP2112K-3.3

Commit message: fix(hardware): correct U3 GND, add fiducials, fix +VRAW via geometry
- Replace U3 pin 3 PWR_FLAG with GND power symbol; buck now has proper
  GND return through the pour instead of floating on Net-(U3-GND)
- Update PCB from schematic to propagate net changes (K1-K12 coil pins,
  U3 tab pad)
- Route +VRAW at Power netclass, complete U3 OUT -> D3-K -> L1-1
  switch node
- Add 3 fiducials (Fiducial_1mm_Mask3mm, Level A) at TR/BL/BR corners
  for PCBA optical alignment; asymmetric layout for orientation
- Fix +VRAW vias: swap diameter/hole (were 0.4/0.8, corrected to 0.8/0.4)
- DRC clean: 0 errors, 0 warnings, 0 unconnected items
Connections:
- net GND: now also C6.2, U3.3 (GND)
Changed lines of the file:
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@@
 	)
 	(junction
-		(at 179.07 54.61)
-		(diameter 0)
-		(color 0 0 0 0)
-	)
-	(junction
 		(at 297.18 58.42)
 		(diameter 0)
@@
 	(wire
 		(pts
-			(xy 179.07 54.61) (xy 181.61 54.61)
-		)
-		(stroke
-			(width 0)
-			(type default)
-		)
-	)
-	(wire
-		(pts
 			(xy 64.77 50.8) (xy 64.77 53.34)
 		)
@@
 	(wire
 		(pts
-			(xy 157.48 54.61) (xy 179.07 54.61)
-		)
-		(stroke
-			(width 0)
-			(type default)
-		)
-	)
-	(wire
-		(pts
 			(xy 46.99 248.92) (xy 54.61 248.92)
 		)
@@
 	)
 	(symbol
+		(lib_id "power:GND")
+		(at 181.61 54.61 0)
+		(unit 1)
+		(body_style 1)
+		(exclude_from_sim no)
+		(in_bom yes)
+		(on_board yes)
+		(in_pos_files yes)
+		(dnp no)
+		(property "Reference" "#PWR040"
+			(at 181.61 60.96 0)
+			(hide yes)
+			(show_name no)
+			(do_not_autoplace no)
+			(effects
+				(font
+					(size 1.27 1.27)
+				)
+			)
+		)
+		(property "Value" "GND"
+			(at 184.15 57.15 0)
+			(show_name no)
+			(do_not_autoplace no)
+			(effects
+				(font
+					(size 1.27 1.27)
+				)
+			)
+		)
+		(property "Footprint" ""
+			(at 181.61 54.61 0)
+			(hide yes)
+			(show_name no)
+			(do_not_autoplace no)
+			(effects
+				(font
+					(size 1.27 1.27)
+				)
+			)
+		)
+		(property "Datasheet" ""
+			(at 181.61 54.61 0)
+			(hide yes)
+			(show_name no)
+			(do_not_autoplace no)
+			(effects
+				(font
+					(size 1.27 1.27)
+				)
+			)
+		)
+		(property "Description" "Power symbol creates a global label with name \"GND\" , ground"
+			(at 181.61 54.61 0)
+			(hide yes)
+			(show_name no)
+			(do_not_autoplace no)
+			(effects
+				(font
+					(size 1.27 1.27)
+				)
+			)
+		)
+		(pin "1"
+		)
+		(instances
+			(project "main-controller-v1"
+				(path "/b1003c9b-a76b-4da0-bb38-3ef06d0104bf"
+					(reference "#PWR040")
+					(unit 1)
+				)
+			)
+		)
+	)
+	(symbol
 		(lib_id "power:+3V3")
 		(at 99.06 96.52 0)
@@
 	)
 	(symbol
-		(lib_id "power:PWR_FLAG")
-		(at 179.07 54.61 180)
-		(unit 1)
-		(body_style 1)
-		(exclude_from_sim no)
-		(in_bom yes)
-		(on_board yes)
-		(in_pos_files yes)
-		(dnp no)
-		(fields_autoplaced yes)
-		(property "Reference" "#FLG02"
-			(at 179.07 56.515 0)
-			(hide yes)
-			(show_name no)
-			(do_not_autoplace no)
-			(effects
-				(font
-					(size 1.27 1.27)
-				)
-			)
-		)
-		(property "Value" "PWR_FLAG"
-			(at 179.07 59.69 0)
-			(show_name no)
-			(do_not_autoplace no)
-			(effects
-				(font
-					(size 1.27 1.27)
-				)
-			)
-		)
-		(property "Footprint" ""
-			(at 179.07 54.61 0)
-			(hide yes)
-			(show_name no)
-			(do_not_autoplace no)
-			(effects
-				(font
-					(size 1.27 1.27)
-				)
-			)
-		)
-		(property "Datasheet" ""
-			(at 179.07 54.61 0)
-			(hide yes)
-			(show_name no)
-			(do_not_autoplace no)
-			(effects
-				(font
-					(size 1.27 1.27)
-				)
-			)
-		)
-		(property "Description" "Special symbol for telling ERC where power comes from"
-			(at 179.07 54.61 0)
-			(hide yes)
-			(show_name no)
-			(do_not_autoplace no)
-			(effects
-				(font
-					(size 1.27 1.27)
-				)
-			)
-		)
-		(pin "1"
-		)
-		(instances
-			(project "main-controller-v1"
-				(path "/b1003c9b-a76b-4da0-bb38-3ef06d0104bf"
-					(reference "#FLG02")
-					(unit 1)
-				)
-			)
-		)
-	)
-	(symbol
 		(lib_id "power:GND")
 		(at 336.55 110.49 0)
@@
 					(unit 1)
 				)
+			)
+		)
+	)
+	(symbol
+		(lib_id "power:GND")
+		(at 157.48 54.61 0)
+		(unit 1)
+		(body_style 1)
+		(exclude_from_sim no)
+		(in_bom yes)
+		(on_board yes)
+		(in_pos_files yes)
+		(dnp no)
+		(property "Reference" "#PWR041"
+			(at 157.48 60.96 0)
+			(hide yes)
+			(show_name no)
+			(do_not_autoplace no)
+			(effects
+				(font
+					(size 1.27 1.27)
+				)
+			)
+		)
+		(property "Value" "GND"
+			(at 160.02 57.15 0)
+			(show_name no)
+			(do_not_autoplace no)
+			(effects
+				(font
+					(size 1.27 1.27)
+				)
+			)
+		)
+		(property "Footprint" ""
+			(at 157.48 54.61 0)
+			(hide yes)
+			(show_name no)
+			(do_not_autoplace no)
+			(effects
+				(font
+					(size 1.27 1.27)
+				)
+			)
+		)
+		(property "Datasheet" ""
+			(at 157.48 54.61 0)
+			(hide yes)
+			(show_name no)
+			(do_not_autoplace no)
+			(effects
+				(font
+					(size 1.27 1.27)
+				)
+			)
+		)
+		(property "Description" "Power symbol creates a global label with name \"GND\" , ground"
+			(at 157.48 54.61 0)
+			(hide yes)
+			(show_name no)
+			(do_not_autoplace no)
+			(effects
+				(font
+					(size 1.27 1.27)
+				)
+			)
+		)
+		(pin "1"
+		)
+		(instances
+			(project "main-controller-v1"
+				(path "/b1003c9b-a76b-4da0-bb38-3ef06d0104bf"
+					(reference "#PWR041")
+					(unit 1)
+				)

Commit message: feat(hardware): rev2 schematic — J1 rewire + power-tree bring-up jumpers
- Rewire J1 (USB-C header) to match B0D962KHF2 pigtail:
  pin1=VBUS, pin2=D-, pin3=D+, pin4=CC1, pin5=CC2, pin6=GND.
  SS14 stays on pin1, 5.1k CC pulldowns on pins 4/5.
- Add R_JMP1-R_JMP4 (0 ohm 1206) as staged bring-up jumpers:
  JMP_AC   (F1 -> D2), JMP_VRAW (+VRAW -> U3.VIN),
  JMP_5V   (U3 out -> +5V), JMP_3V3 (U4 out -> +3V3).
- Move C6 to buck side of R_JMP2 to decouple U3.VIN locally.
- Add PWR_FLAG on downstream +3V3 rail for ERC.
- ERC clean.

Refs: rev2 punch list #21, #25.
Parts:
- removed J1: USB_C_Receptacle_USB2.0_16P, Connector_USB:USB_C_Receptacle_HRO_TYPE-C-31-M-12, symbol Connector:USB_C_Receptacle_USB2.0_16P
- added FID1, FID2, FID3: Fiducial, Fiducial:Fiducial_1mm_Mask2mm, symbol Mechanical:Fiducial
- added J1: B6B-PH-K-S, Connector_JST:JST_PH_B6B-PH-K_1x06_P2.00mm_Vertical, symbol Connector_Generic:Conn_01x06
- added R_JMP1, R_JMP2, R_JMP3, R_JMP4: 0, symbol Device:R
- C1, C8, C9: LCSC (none) -> C15850
- C10, C11, C2, C4: LCSC (none) -> C14663
- C3: LCSC (none) -> C15849
- C5, D3, J2, J3, J4, J6, SW1, SW2: now not fitted
- C6: LCSC (none) -> C2836438
- C7: LCSC (none) -> C178541
- D1: LCSC (none) -> C78420
- D2: LCSC (none) -> C5377
- D4: LCSC (none) -> C2480
- D5: LCSC (none) -> C2761795
- F1: LCSC (none) -> C17313
- K1, K10, K11, K12, K2, K3, K4, K5, K6, K7, K8, K9: LCSC (none) -> C401984
- L1: LCSC (none) -> C840528
- R1, R2, R5, R6: LCSC (none) -> C25804
- R10, R11, R12, R13, R14, R15, R16, R17, R18, R7, R8, R9: LCSC (none) -> C23138
- R3, R4: LCSC (none) -> C23186
- U1: LCSC (none) -> C2913204
- U2: LCSC (none) -> C7519
- U3: LCSC (none) -> C5276750
- U4: LCSC (none) -> C51118
Connections:
- net +3V3: now also R_JMP4.2; no longer C10.1, C9.2, U4.5 (VOUT)
- net +5V: now also R_JMP3.1; no longer C7.1, L1.2, U3.4 (FB)
- net +VRAW: now also D1.2 (A2), D2.4 (+), R_JMP2.1; no longer C6.1, D2.1 (+), U3.1 (VIN)
- net 24VAC_COM: now also D2.3; no longer D1.1 (A1), D2.4
- net 24VAC_HOT: now also D2.1; no longer D1.2 (A2), D2.3
- net GND: now also D1.1 (A1), J1.6 (Pin_6)
- net USB_D+_RAW: now also J1.3 (Pin_3)
- net USB_D-_RAW: now also J1.2 (Pin_2)
- net at D4.2 (A): now also J1.1 (Pin_1)
- net at R3.1: now also J1.4 (Pin_4)
- net at R4.1: now also J1.5 (Pin_5)
- net at J2.1 (Pin_1): now also R_JMP1.2; no longer F1.2
- new net: F1.2, R_JMP1.1
- new net: C10.1, C9.2, R_JMP4.1, U4.5 (VOUT)
- new net: C7.1, L1.2, R_JMP3.2, U3.4 (FB)
- new net: C6.1, R_JMP2.2, U3.1 (VIN)
- no-connect marks 21 -> 19
Other:
- note added: "USB-C Header"
- note removed: "USB-C Port"
- moved on the sheet: C6, D1, D4, F1, R3, R4

Commit message: fix(hardware): replace D2 bridge rectifier with MB10S, add bring-up jumpers, C7 footprint fix
- D2: DB107S (C5377, Extended) → MB10S (C2488, Basic); symbol+footprint
  imported via easyeda2kicad, DFM-authoritative pinout resolves the D2
  pad-swap risk that killed rev1 confidence
- Add R_JMP1-4 (0Ω 1206) on 24VAC_HOT, +VRAW, +5V, +3V3 for per-rail
  current measurement during bring-up
- C7 footprint: CP_Elec_6.3x5.4 → CP_Elec_5x5.8 (matches purchased part)
- Regenerate production/ gerbers, BOM, and CPL to match
- Track Azul.kicad_sym + Azul.pretty/MBS_* + Azul.3dshapes/ + sym-lib-table
  so the schematic resolves on a fresh clone
- Save datasheets for rev2 triac stage (MOC3062M, BT137-600E) and the
  G3MB-202P EOL catalog from Yuke Chip
Parts:
- removed D2: DB107S, Diode_SMD:Diode_Bridge_Diotec_SO-DIL-Slim, symbol Device:D_Bridge_+-AA
- added D2: MB10S_C2488, Azul:MBS_L4.7-W3.8-P2.40-LS7.0-TL, symbol Azul:MB10S_C2488
- C7: footprint Capacitor_SMD:CP_Elec_6.3x5.4 -> Capacitor_SMD:CP_Elec_5x5.8
- J1: now not fitted
- R_JMP1, R_JMP2, R_JMP3, R_JMP4: footprint (none) -> Resistor_SMD:R_1206_3216Metric; LCSC (none) -> C17168
Connections:
- net +VRAW: now also D2.1 (+)
- net 24VAC_COM: now also D2.3 (C2)
- net 24VAC_HOT: now also D2.4 (C1)
- net GND: now also D2.2 (-)
Other:
- moved on the sheet: C10, C4, C5, C6, C7, C8, C9, D1, D3, D4, F1, J2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

Commit message: feat(hardware): rev2 fab package — 12× discrete triac zone drivers
Rev2 replaces the EOL Omron G3MB-202P SSRs with a discrete triac zone-
driver topology (MOC3062M opto-isolated zero-cross trigger → BT137-600E
triac, per-zone snubber and X2 line cap). Twelve identical zone-driver
hierarchical sheets fan out from the parent under a single ribbon
header, driven active-high from the WROOM GPIOs.

Fab package uploaded to JLC 2026-08-08 as order W2026080821415396
(5 boards, Standard PCBA, UPS Express DDP, ~2026-08-18 delivery).

Design changes
- Delete K1–K12 G3MB relays; instantiate zone-driver.kicad_sch × 12
- Renumber R/C/U/Q across all 12 zone sheets (Q1–Q12 triacs,
  U5–U16 opto-drivers, C12–C23 X2 caps, R7–R42 zone stage)
- parts.yaml rev2 BOM: BT137-600E C967624, MOC3062M C8919,
  10nF X2 C105755, 39Ω 2010 snubber C2692665
- New Azul.pretty footprints + 3D models for DIP-6 opto, TO-220
  triac, and CAP-TH X2 (10mm pitch)
- Silkscreen title block "Rev 2 · 2026-08"

Fab workflow tooling
- scripts/apply_lcsc_fields.py: patches .kicad_sch LCSC fields from
  parts.yaml (BOM source of truth)
- jlc-dnp-lookup.md: fate: dnp vs smt decision matrix per part
- JLC_UPLOAD_TRACKER.md: 5-step walkthrough incorporating rev1
  lessons (J1 orientation, D2 pad-swap, CPL rotation offsets)
- Fixed DNP-flag sync bug — direct .kicad_pcb (attr) edit to strip
  stale dnp from J2/J3/J4 after fate: dnp→smt flip

Datasheets committed under docs/hardware/ for all rev2-new Extended
parts (C105755 X2, C2692665 39Ω 2010, C5188434 MX126 terminal,
C3817964, C6947975).

.gitignore: filter kicad-cli export intermediates (*.pre-*-backup,
DRC-output.rpt, update-pcb-report.txt) and the docs/azul v1 - Omega/
reference dump.
Parts:
- removed K1, K10, K11, K12, K2, K3, K4, K5, K6, K7, K8, K9: G3MB-202P, Azul:G3MB-202P, symbol Azul:G3MB-202P
- removed R10, R11, R12, R13, R14, R15, R16, R17, R18, R7, R8, R9: 330, Resistor_SMD:R_0603_1608Metric, symbol Device:R_Small
- J2, J3, J4: LCSC (none) -> C5188434; now fitted
Connections:
- net ZONE1: now also U1.31 (GPIO38/FSPIWP/SUBSPIWP); no longer U1.6 (GPIO6/TOUCH6/ADC1_CH5)
- net ZONE11: now also U1.7 (GPIO7/TOUCH7/ADC1_CH6); no longer U1.11 (GPIO18/U1RXD/ADC2_CH7/CLK_OUT3)
- net ZONE12: now also U1.6 (GPIO6/TOUCH6/ADC1_CH5); no longer U1.31 (GPIO38/FSPIWP/SUBSPIWP)
- net ZONE2: now also U1.22 (GPIO14/TOUCH14/ADC2_CH3/FSPIWP/FSPIDQS/SUBSPIWP); no longer U1.7 (GPIO7/TOUCH7/ADC1_CH6)
- net ZONE3: now also U1.21 (GPIO13/TOUCH13/ADC2_CH2/FSPIQ/FSPIIO7/SUBSPIQ); no longer U1.12 (GPIO8/TOUCH8/ADC1_CH7/SUBSPICS1)
- net ZONE4: now also U1.20 (GPIO12/TOUCH12/ADC2_CH1/FSPICLK/FSPIIO6/SUBSPICLK); no longer U1.17 (GPIO9/TOUCH9/ADC1_CH8/FSPIHD/SUBSPIHD)
- net ZONE5: now also U1.19 (GPIO11/TOUCH11/ADC2_CH0/FSPID/FSPIIO5/SUBSPID); no longer U1.18 (GPIO10/TOUCH10/ADC1_CH9/FSPICS0/FSPIIO4/SUBSPICS0)
- net ZONE6: now also U1.18 (GPIO10/TOUCH10/ADC1_CH9/FSPICS0/FSPIIO4/SUBSPICS0); no longer U1.19 (GPIO11/TOUCH11/ADC2_CH0/FSPID/FSPIIO5/SUBSPID)
- net ZONE7: now also U1.17 (GPIO9/TOUCH9/ADC1_CH8/FSPIHD/SUBSPIHD); no longer U1.20 (GPIO12/TOUCH12/ADC2_CH1/FSPICLK/FSPIIO6/SUBSPICLK)
- net ZONE8: now also U1.12 (GPIO8/TOUCH8/ADC1_CH7/SUBSPICS1); no longer U1.21 (GPIO13/TOUCH13/ADC2_CH2/FSPIQ/FSPIIO7/SUBSPIQ)
- net ZONE9: now also U1.11 (GPIO18/U1RXD/ADC2_CH7/CLK_OUT3); no longer U1.22 (GPIO14/TOUCH14/ADC2_CH3/FSPIWP/FSPIDQS/SUBSPIWP)
Other:
- added sheet zone1 (zone-driver.kicad_sch)
- added sheet zone10 (zone-driver.kicad_sch)
- added sheet zone11 (zone-driver.kicad_sch)
- added sheet zone12 (zone-driver.kicad_sch)
- added sheet zone2 (zone-driver.kicad_sch)
- added sheet zone3 (zone-driver.kicad_sch)
- added sheet zone4 (zone-driver.kicad_sch)
- added sheet zone5 (zone-driver.kicad_sch)
- added sheet zone6 (zone-driver.kicad_sch)
- added sheet zone7 (zone-driver.kicad_sch)
- added sheet zone8 (zone-driver.kicad_sch)
- added sheet zone9 (zone-driver.kicad_sch)
